File: pcb/watch.kicad_sch (KiCad schematic)
At the start: 26 parts, among them SW1 EVP-AA202K, SW2 EVP-AA202K, U1 ATtiny402-SS

Commit message: Use a CR2032 instead of a CR1216
Parts:
- removed BT1: BK-916-TR, BAT_BK-916-TR, symbol Battery Holder:BK-916-TR
- added BT1: BAT-HLD-001-TR, Battery Holder:BAT_BAT-HLD-001-TR, symbol Battery Holder:BAT-HLD-001-TR
- added TP4: TestPoint, TestPoint:TestPoint_Pad_D1.0mm, symbol Connector:TestPoint
- R5, R6: value 4.7 kΩ -> 10 kΩ
Connections:
- net +3.3V: now also BT1.P1, BT1.P2
- net GND: now also BT1.N1
- net at D1.2 (A), D11.2 (A), D12.1 (K)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: now also TP4.1
Changed lines of the file:
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@@
+    (stroke (width 0) (type default) (color 0 0 0 0))
+  )
+  (wire (pts (xy 64.77 81.28) (xy 64.77 86.36))
     (stroke (width 0) (type default) (color 0 0 0 0))
   )
@@
     (stroke (width 0) (type default) (color 0 0 0 0))
   )
-  (wire (pts (xy 64.77 97.79) (xy 64.77 100.33))
+  (wire (pts (xy 64.77 101.6) (xy 64.77 106.68))
     (stroke (width 0) (type default) (color 0 0 0 0))
   )
@@
     (stroke (width 0) (type default) (color 0 0 0 0))
   )
+  (wire (pts (xy 153.67 46.99) (xy 153.67 50.8))
+    (stroke (width 0) (type default) (color 0 0 0 0))
+  )
   (wire (pts (xy 144.78 101.6) (xy 144.78 114.3))
     (stroke (width 0) (type default) (color 0 0 0 0))
@@
   )
   (wire (pts (xy 176.53 50.8) (xy 176.53 53.34))
-    (stroke (width 0) (type default) (color 0 0 0 0))
-  )
-  (wire (pts (xy 64.77 85.09) (xy 64.77 87.63))
     (stroke (width 0) (type default) (color 0 0 0 0))
   )
@@
     (pin "2")
   )
-  (symbol (lib_id "Battery Holder:BK-916-TR") (at 64.77 92.71 90) (unit 1)
-    (in_bom yes) (on_board yes) (fields_autoplaced)
-    (property "Reference" "BT1" (id 0) (at 68.58 91.4399 90)
-      (effects (font (size 1.27 1.27)) (justify right))
-    )
-    (property "Value" "BK-916-TR" (id 1) (at 68.58 93.9799 90)
-      (effects (font (size 1.27 1.27)) (justify right))
-    )
-    (property "Footprint" "BAT_BK-916-TR" (id 2) (at 64.77 92.71 0)
-      (effects (font (size 1.27 1.27)) (justify bottom) hide)
-    )
-    (property "Datasheet" "" (id 3) (at 64.77 92.71 0)
-      (effects (font (size 1.27 1.27)) hide)
-    )
-    (property "PARTREV" "A" (id 4) (at 64.77 92.71 0)
-      (effects (font (size 1.27 1.27)) (justify bottom) hide)
-    )
-    (property "STANDARD" "MANUFACTURER RECOMMENDATIONS" (id 5) (at 64.77 92.71 0)
-      (effects (font (size 1.27 1.27)) (justify bottom) hide)
-    )
-    (property "MANUFACTURER" "Memory Protection Devices INC" (id 6) (at 64.77 92.71 0)
-      (effects (font (size 1.27 1.27)) (justify bottom) hide)
-    )
-    (pin "1")
-    (pin "2")
-    (pin "3")
-  )
   (symbol (lib_id "power:GND") (at 114.3 35.56 0) (unit 1)
     (in_bom yes) (on_board yes) (fields_autoplaced)
@@
     )
     (pin "1")
+  )
+  (symbol (lib_id "Connector:TestPoint") (at 153.67 46.99 0) (unit 1)
+    (in_bom yes) (on_board yes) (fields_autoplaced)
+    (property "Reference" "TP4" (id 0) (at 156.21 43.6879 0)
+      (effects (font (size 1.27 1.27)) (justify left))
+    )
+    (property "Value" "TestPoint" (id 1) (at 154.9399 41.91 90)
+      (effects (font (size 1.27 1.27)) (justify left) hide)
+    )
+    (property "Footprint" "TestPoint:TestPoint_Pad_D1.0mm" (id 2) (at 158.75 46.99 0)
+      (effects (font (size 1.27 1.27)) hide)
+    )
+    (property "Datasheet" "~" (id 3) (at 158.75 46.99 0)
+      (effects (font (size 1.27 1.27)) hide)
+    )
+    (pin "1")
+  )
+  (symbol (lib_id "Battery Holder:BAT-HLD-001-TR") (at 64.77 93.98 270) (unit 1)
+    (in_bom yes) (on_board yes) (fields_autoplaced)
+    (property "Reference" "BT1" (id 0) (at 68.58 92.0749 90)
+      (effects (font (size 1.27 1.27)) (justify left))
+    )
+    (property "Value" "BAT-HLD-001-TR" (id 1) (at 68.58 94.6149 90)
+      (effects (font (size 1.27 1.27)) (justify left))
+    )
+    (property "Footprint" "Battery Holder:BAT_BAT-HLD-001-TR" (id 2) (at 64.77 93.98 0)
+      (effects (font (size 1.27 1.27)) (justify bottom) hide)
+    )
+    (property "Datasheet" "" (id 3) (at 64.77 93.98 0)
+      (effects (font (size 1.27 1.27)) hide)
+    )
+    (property "PARTREV" "B" (id 4) (at 64.77 93.98 0)
+      (effects (font (size 1.27 1.27)) (justify bottom) hide)
+    )
+    (property "STANDARD" "Manufacturer Recommendations" (id 5) (at 64.77 93.98 0)
+      (effects (font (size 1.27 1.27)) (justify bottom) hide)
+    )
+    (property "MAXIMUM_PACKAGE_HEIGHT" "4.2 mm" (id 6) (at 64.77 93.98 0)
+      (effects (font (size 1.27 1.27)) (justify bottom) hide)
+    )
+    (property "MANUFACTURER" "Linx Technologies" (id 7) (at 64.77 93.98 0)
+      (effects (font (size 1.27 1.27)) (justify bottom) hide)
+    )
+    (pin "N1")
+    (pin "P1")
+    (pin "P2")
   )
   (symbol (lib_id "Device:R_Small_US") (at 105.41 45.72 90) (unit 1)
@@
     (pin "2")
   )
-  (symbol (lib_id "power:GND") (at 64.77 100.33 0) (unit 1)
-    (in_bom yes) (on_board yes) (fields_autoplaced)
-    (property "Reference" "#PWR0107" (id 0) (at 64.77 106.68 0)
-      (effects (font (size 1.27 1.27)) hide)
-    )
-    (property "Value" "GND" (id 1) (at 64.77 105.41 0))
-    (property "Footprint" "" (id 2) (at 64.77 100.33 0)
-      (effects (font (size 1.27 1.27)) hide)
-    )
-    (property "Datasheet" "" (id 3) (at 64.77 100.33 0)
+  (symbol (lib_id "power:GND") (at 64.77 106.68 0) (unit 1)
+    (in_bom yes) (on_board yes) (fields_autoplaced)
+    (property "Reference" "#PWR0107" (id 0) (at 64.77 113.03 0)
+      (effects (font (size 1.27 1.27)) hide)
+    )
+    (property "Value" "GND" (id 1) (at 64.77 111.76 0))
+    (property "Footprint" "" (id 2) (at 64.77 106.68 0)
+      (effects (font (size 1.27 1.27)) hide)
+    )
+    (property "Datasheet" "" (id 3) (at 64.77 106.68 0)
       (effects (font (size 1.27 1.27)) hide)
     )
@@
       (effects (font (size 1.27 1.27)) (justify left))
     )
-    (property "Value" "4.7 kΩ" (id 1) (at 147.32 97.7899 0)
+    (property "Value" "10 kΩ" (id 1) (at 147.32 97.7899 0)
       (effects (font (size 1.27 1.27)) (justify left))
     )
@@
       (effects (font (size 1.27 1.27)) (justify left))
     )
-    (property "Value" "4.7 kΩ" (id 1) (at 151.13 132.0799 0)
+    (property "Value" "10 kΩ" (id 1) (at 151.13 132.0799 0)
       (effects (font (size 1.27 1.27)) (justify left))
     )
@@
     (pin "4")
   )
-  (symbol (lib_id "power:+3.3V") (at 64.77 85.09 0) (unit 1)
-    (in_bom yes) (on_board yes) (fields_autoplaced)
-    (property "Reference" "#PWR0106" (id 0) (at 64.77 88.9 0)
-      (effects (font (size 1.27 1.27)) hide)
-    )
-    (property "Value" "+3.3V" (id 1) (at 64.77 80.01 0))
-    (property "Footprint" "" (id 2) (at 64.77 85.09 0)
-      (effects (font (size 1.27 1.27)) hide)
-    )
-    (property "Datasheet" "" (id 3) (at 64.77 85.09 0)
+  (symbol (lib_id "power:+3.3V") (at 64.77 81.28 0) (unit 1)
+    (in_bom yes) (on_board yes) (fields_autoplaced)
+    (property "Reference" "#PWR0106" (id 0) (at 64.77 85.09 0)
+      (effects (font (size 1.27 1.27)) hide)
+    )
+    (property "Value" "+3.3V" (id 1) (at 64.77 76.2 0))
+    (property "Footprint" "" (id 2) (at 64.77 81.28 0)
+      (effects (font (size 1.27 1.27)) hide)
+    )
+    (property "Datasheet" "" (id 3) (at 64.77 81.28 0)
       (effects (font (size 1.27 1.27)) hide)
     )
@@
       (reference "#PWR0108") (unit 1) (value "+3.3V") (footprint "")
     )
-    (path "/1beb004e-f400-4728-bfe5-a2d9dc5faf02"
-      (reference "BT1") (unit 1) (value "BK-916-TR") (footprint "BAT_BK-916-TR")
+    (path "/306d5627-4898-4c6f-83bd-7f9ef5e03fa3"
+      (reference "BT1") (unit 1) (value "BAT-HLD-001-TR") (footprint "Battery Holder:BAT_BAT-HLD-001-TR")
     )
     (path "/69e545a7-e731-4e30-a3f4-1d38db51a067"
@@
     )
     (path "/ca594061-c91d-408d-b372-c919964b5c34"
-      (reference "R5") (unit 1) (value "4.7 kΩ") (footprint "Resistor_SMD:R_0603_1608Metric")
+      (reference "R5") (unit 1) (value "10 kΩ") (footprint "Resistor_SMD:R_0603_1608Metric")
     )
     (path "/d68fff31-8e4a-4485-bfbb-aecad0461d56"
-      (reference "R6") (unit 1) (value "4.7 kΩ") (footprint "Resistor_SMD:R_0603_1608Metric")
+      (reference "R6") (unit 1) (value "10 kΩ") (footprint "Resistor_SMD:R_0603_1608Metric")
     )
     (path "/3a1d0747-9e6f-4d73-8e44-3a3850d9d1a1"
@@
       (reference "TP3") (unit 1) (value "TestPoint") (footprint "TestPoint:TestPoint_Pad_1.0x1.0mm")
     )
+    (path "/2e484d8a-7739-49d7-a241-c70c7dfa7238"
+      (reference "TP4") (unit 1) (value "TestPoint") (footprint "TestPoint:TestPoint_Pad_D1.0mm")
+    )
     (path "/5cff94aa-a71d-4632-a264-71f194704450"
